File: KiCAD/gearclock.sch (KiCad schematic (older format))
At the start: 44 parts, among them J1 SW_EXT, P1 ISP, P10 I/O, P11 GPS, P12 BAT, P13 LiPo, P2 FTDI, P3 CD1, P4 CD2, P5 MOTOR, P6 MOTOR_R, P7 MOTOR_L, P8 I/O, P9 I/O, SW1 RST, SW2 SW_UP, SW3 SW_DN, SW4 SW_OK, SW5 SW_LT, SW6 SW_RT, U1 ATMEGA328P, U2 Hall_Sensor, U3 3V3, X1 8MHz

Commit message: review the schematic
Parts:
- added C?: 100n, C4_Pretty:c_0805_led, symbol C
Connections:
- net +3.3V: now also C?.1
- net GND: now also C?.2
- net LED2 renamed LED1
Other:
- moved on the sheet: B1, C5, LED1, R4
Changed lines of the file:
@@
 	3400 4050 3625 4050
 Wire Wire Line
-	3400 3850 5975 3850
+	3400 3850 6225 3850
 Wire Wire Line
 	3400 3750 3625 3750
@@
 L R R4
 U 1 1 4DCFFAF9
-P 5975 2975
-F 0 "R4" H 5875 3100 50  0000 C CNN
-F 1 "750E" V 5975 2975 40  0000 C CNN
-F 2 "ArthurC Lib:r_0805" H 5975 2975 60  0001 C CNN
-F 3 "" H 5975 2975 60  0001 C CNN
-	1    5975 2975
+P 6225 2975
+F 0 "R4" H 6125 3100 50  0000 C CNN
+F 1 "750E" V 6225 2975 40  0000 C CNN
+F 2 "ArthurC Lib:r_0805" H 6225 2975 60  0001 C CNN
+F 3 "" H 6225 2975 60  0001 C CNN
+	1    6225 2975
 	1    0    0    -1
 $EndComp
@@
 Text Label 3625 2450 0    40   ~ 0
 M1
-Text Label 3450 2950 0    40   ~ 0
+Text Label 3625 2950 0    40   ~ 0
 Hall
 Text Label 3625 3150 0    40   ~ 0
@@
 Text Label 3625 3350 0    40   ~ 0
 1pps
-Text Label 3450 3850 0    40   ~ 0
-LED2
+Text Label 3625 3850 0    40   ~ 0
+LED1
 Text Label 3625 3550 0    40   ~ 0
 STP
@@
 	1    0    0    -1
 $EndComp
-Text Label 3450 2650 0    40   ~ 0
+Text Label 3625 2650 0    40   ~ 0
 SDA
-Text Label 3450 2750 0    40   ~ 0
+Text Label 3625 2750 0    40   ~ 0
 SCL
 Text Label 2575 1100 0    60   ~ 0
@@
 Text Label 5350 4900 0    40   ~ 0
 GND
-Text Label 3450 4250 0    40   ~ 0
+Text Label 3625 4250 0    40   ~ 0
 SS
-Text Label 3450 4350 0    40   ~ 0
+Text Label 3625 4350 0    40   ~ 0
 MOSI
-Text Label 3450 4550 0    40   ~ 0
+Text Label 3625 4550 0    40   ~ 0
 SCK
-Text Label 3450 4450 0    40   ~ 0
+Text Label 3625 4450 0    40   ~ 0
 MISO
 $Comp
@@
 U 1 1 54D79F22
 P 5100 1950
-F 0 "U2" H 5225 1875 40  0000 L CNN
-F 1 "Hall_Sensor" H 5225 1800 40  0000 L CNN
+F 0 "U2" H 4900 2075 40  0000 L CNN
+F 1 "Hall_Sensor" V 5250 1775 40  0000 L CNN
 F 2 "" H 5100 2100 60  0000 C CNN
 F 3 "" H 5100 2100 60  0000 C CNN
@@
 L C C5
 U 1 1 54ECC15D
-P 6450 1600
-F 0 "C5" H 6475 1700 50  0000 L CNN
-F 1 "100n" H 6475 1500 50  0000 L CNN
-F 2 "C4_Pretty:c_0805_led" H 6450 1600 50  0001 C CNN
-F 3 "" H 6450 1600 60  0001 C CNN
-F 4 "CAP CER 0.1UF 25V 10% X7R 0805" H 6450 1800 60  0001 L CNN "Field4"
-F 5 "100nF, 25V" H 6450 1900 60  0001 L CNN "Field5"
-F 6 "Surface Mount, MLCC" H 6450 2000 60  0001 L CNN "Field6"
-F 7 "Kemet" H 6450 2100 60  0001 L CNN "Field7"
-F 8 "C0805C104K3RACTU" H 6450 2200 60  0001 L CNN "Field8"
-F 9 "Digikey" H 6450 2300 60  0001 L CNN "Field9"
-F 10 "399-1168-1-ND" H 6450 2400 60  0001 L CNN "Field10"
-F 11 "http://www.digikey.com/product-detail/en/C0805C104K3RACTU/399-1168-1-ND/411443" H 6450 2500 60  0001 L CNN "Field11"
-	1    6450 1600
+P 6700 1600
+F 0 "C5" H 6725 1700 50  0000 L CNN
+F 1 "100n" H 6725 1500 50  0000 L CNN
+F 2 "C4_Pretty:c_0805_led" H 6700 1600 50  0001 C CNN
+F 3 "" H 6700 1600 60  0001 C CNN
+F 4 "CAP CER 0.1UF 25V 10% X7R 0805" H 6700 1800 60  0001 L CNN "Field4"
+F 5 "100nF, 25V" H 6700 1900 60  0001 L CNN "Field5"
+F 6 "Surface Mount, MLCC" H 6700 2000 60  0001 L CNN "Field6"
+F 7 "Kemet" H 6700 2100 60  0001 L CNN "Field7"
+F 8 "C0805C104K3RACTU" H 6700 2200 60  0001 L CNN "Field8"
+F 9 "Digikey" H 6700 2300 60  0001 L CNN "Field9"
+F 10 "399-1168-1-ND" H 6700 2400 60  0001 L CNN "Field10"
+F 11 "http://www.digikey.com/product-detail/en/C0805C104K3RACTU/399-1168-1-ND/411443" H 6700 2500 60  0001 L CNN "Field11"
+	1    6700 1600
 	1    0    0    -1
 $EndComp
@@
 L WS2812B LED1
 U 1 1 54ECC16E
-P 5900 1975
-F 0 "LED1" H 5800 1500 40  0000 C CNN
-F 1 "WS2812B" V 5775 1950 40  0000 C CNN
-F 2 "C4_Pretty:RGB_WS2811B" H 5900 1975 60  0001 C CNN
-F 3 "~" H 5900 1975 60  0000 C CNN
-	1    5900 1975
+P 6150 1975
+F 0 "LED1" H 6050 1500 40  0000 C CNN
+F 1 "WS2812B" V 6025 1950 40  0000 C CNN
+F 2 "C4_Pretty:RGB_WS2811B" H 6150 1975 60  0001 C CNN
+F 3 "~" H 6150 1975 60  0000 C CNN
+	1    6150 1975
 	1    0    0    1
 $EndComp
@@
 3V3
 Wire Wire Line
-	6175 1350 6175 1100
-Connection ~ 6175 1100
-Wire Wire Line
-	5975 2550 5975 2725
-Wire Wire Line
-	5975 3850 5975 3225
-Wire Wire Line
-	6450 1400 6450 1250
-Wire Wire Line
-	6450 1250 6175 1250
-Connection ~ 6175 1250
-Wire Wire Line
-	6450 1800 6450 1950
-Wire Wire Line
-	5975 1350 5975 1250
-Wire Wire Line
-	5975 1250 5475 1250
-Wire Wire Line
-	5475 1250 5475 1550
+	6425 1100 6425 1350
+Connection ~ 6425 1100
+Wire Wire Line
+	6225 2550 6225 2725
+Wire Wire Line
+	6225 3850 6225 3225
+Wire Wire Line
+	6700 1400 6700 1250
+Wire Wire Line
+	6700 1250 6425 1250
+Connection ~ 6425 1250
+Wire Wire Line
+	6700 1800 6700 1950
+Wire Wire Line
+	6225 1350 6225 1250
+Wire Wire Line
+	6225 1250 5725 1250
+Wire Wire Line
+	5725 1250 5725 1550
 $Comp
 L GND #PWR09
 U 1 1 54ED6040
-P 5475 1550
-F 0 "#PWR09" H 5475 1550 30  0001 C CNN
-F 1 "GND" H 5475 1480 30  0001 C CNN
-F 2 "" H 5475 1550 60  0001 C CNN
-F 3 "" H 5475 1550 60  0001 C CNN
-	1    5475 1550
+P 5725 1550
+F 0 "#PWR09" H 5725 1550 30  0001 C CNN
+F 1 "GND" H 5725 1480 30  0001 C CNN
+F 2 "" H 5725 1550 60  0001 C CNN
+F 3 "" H 5725 1550 60  0001 C CNN
+	1    5725 1550
 	1    0    0    -1
 $EndComp
@@
 L GND #PWR010
 U 1 1 54ED6076
-P 6450 1950
-F 0 "#PWR010" H 6450 1950 30  0001 C CNN
-F 1 "GND" H 6450 1880 30  0001 C CNN
-F 2 "" H 6450 1950 60  0001 C CNN
-F 3 "" H 6450 1950 60  0001 C CNN
-	1    6450 1950
+P 6700 1950
+F 0 "#PWR010" H 6700 1950 30  0001 C CNN
+F 1 "GND" H 6700 1880 30  0001 C CNN
+F 2 "" H 6700 1950 60  0001 C CNN
+F 3 "" H 6700 1950 60  0001 C CNN
+	1    6700 1950
 	1    0    0    -1
 $EndComp
@@
 L I/O B1
 U 1 1 54ED61D2
-P 6175 2875
-F 0 "B1" H 6255 2875 40  0000 L CNN
-F 1 "I/O" H 6175 2930 30  0001 C CNN
-F 2 "" H 6175 2875 60  0000 C CNN
-F 3 "" H 6175 2875 60  0000 C CNN
-	1    6175 2875
+P 6425 2875
+F 0 "B1" H 6505 2875 40  0000 L CNN
+F 1 "I/O" H 6425 2930 30  0001 C CNN
+F 2 "" H 6425 2875 60  0000 C CNN
+F 3 "" H 6425 2875 60  0000 C CNN
+	1    6425 2875
 	0    1    1    0
 $EndComp
 Wire Wire Line
-	6175 2550 6175 2725
+	6425 2550 6425 2725
 Text Label 3625 2550 0    40   ~ 0
 SW
 Wire Wire Line
 	3625 2550 3400 2550
+$Comp
+L C C?
+U 1 1 5576F5A0
+P 5425 1950
+F 0 "C?" H 5450 2050 50  0000 L CNN
+F 1 "100n" H 5450 1850 50  0000 L CNN
+F 2 "C4_Pretty:c_0805_led" H 5425 1950 50  0001 C CNN
+F 3 "" H 5425 1950 60  0001 C CNN
+F 4 "CAP CER 0.1UF 25V 10% X7R 0805" H 5425 2150 60  0001 L CNN "Field4"
+F 5 "100nF, 25V" H 5425 2250 60  0001 L CNN "Field5"
+F 6 "Surface Mount, MLCC" H 5425 2350 60  0001 L CNN "Field6"
+F 7 "Kemet" H 5425 2450 60  0001 L CNN "Field7"
+F 8 "C0805C104K3RACTU" H 5425 2550 60  0001 L CNN "Field8"
+F 9 "Digikey" H 5425 2650 60  0001 L CNN "Field9"
+F 10 "399-1168-1-ND" H 5425 2750 60  0001 L CNN "Field10"
+F 11 "http://www.digikey.com/product-detail/en/C0805C104K3RACTU/399-1168-1-ND/411443" H 5425 2850 60  0001 L CNN "Field11"
+	1    5425 1950
+	1    0    0    -1
+$EndComp
+Wire Wire Line
+	5425 1750 5425 1600
+Wire Wire Line
+	5425 1600 5100 1600
+Connection ~ 5100 1600
+Wire Wire Line
+	5425 2150 5425 2275
+Wire Wire Line
+	5425 2275 5100 2275
+Connection ~ 5100 2275
 $EndSCHEMATC

Commit message: Schematic, work in progress
Parts:
- removed J1: SW_EXT, PIN_ARRAY_3x1, symbol CONN_3
- removed P1: ISP, ArthurC Lib:ISP, symbol ISP
- removed P11: GPS, ArthurC Lib:PIN_ARRAY-9X1, symbol CONN_9
- removed P12: BAT, ArthurC Lib:pin_strip_2, symbol CONN_2
- removed P13: LiPo, ArthurC Lib:pin_strip_2, symbol CONN_2
- removed P2: FTDI, ArthurC Lib:PIN_ARRAY-6X1, symbol CONN_6
- removed P3: CD1, ArthurC Lib:Sck-04-F-SMT, symbol CONN_4
- removed P4: CD2, ArthurC Lib:Sck-04-F-SMT, symbol CONN_4
- removed P5: MOTOR, symbol CONN_4
- removed P6: MOTOR_R, ArthurC Lib:PIN_ARRAY-6X1, symbol CONN_8
- removed P7: MOTOR_L, ArthurC Lib:PIN_ARRAY-6X1, symbol CONN_8
- added P1: ISP, symbol CONN_02X03
- added P11: GPS, symbol CONN_01X09
- added P12: BAT, symbol CONN_01X02
- added P13: LiPo, symbol CONN_01X02
- added P2: FTDI, symbol CONN_01X06
- added P3: SW_EXT, symbol CONN_01X03
- added P5: Motor, symbol CONN_01X04
- added P6: Motor_R, symbol CONN_01X08
- added P7: Motor_L, symbol CONN_01X08
- U1: symbol ATMEGA8-AI -> ATMEGA328-TQFP32
- gave numbers to parts that had none: 1
Connections:
- net +3.3V: now also P1.2 (P2), P11.8 (P8), P12.1 (P1), P2.3 (P3), P3.1 (P1), P6.6 (P6)
- net 1pps: now also P11.9 (P9)
- net 3Vgps: now also P11.1 (P1)
- net A1: now also P5.3 (P3), P7.5 (P5)
- net A2: now also P5.4 (P4), P7.6 (P6)
- net B1: now also P5.2 (P2), P7.4 (P4)
- net B2: now also P5.1 (P1), P7.3 (P3)
- net BAT: now also P13.2 (P2), P7.1 (P1)
- net CFG: now also P6.4 (P4)
- net DIR: now also P6.8 (P8)
- net EN: now also P6.1 (P1)
- net FIX: now also P11.4 (P4)
- net FLT: now also P7.7 (P7)
- net GND: now also P1.6 (P6), P11.7 (P7), P12.2 (P2), P13.1 (P1), P2.1 (P1), P2.2 (P2), P3.3 (P3), P7.2 (P2), P7.8 (P8)
- net GPS_BAT: now also P11.3 (P3)
- net GPS_EN: now also P11.2 (P2)
- net GPS_Rx: now also P11.6 (P6)
- net GPS_Tx: now also P11.5 (P5)
- net M0: now also P6.2 (P2)
- net M1: now also P6.3 (P3)
- net MISO: now also P1.1 (P1)
- net MOSI: now also P1.4 (P4)
- net RESET: now also P1.5 (P5)
- net RXD: now also P2.4 (P4)
- net SCK: now also P1.3 (P3)
- net STP: now also P6.7 (P7)
- net SW: now also P3.2 (P2)
- net TXD: now also P2.5 (P5)
- net VREF: now also P6.5 (P5)
- net at C4.1: now also P2.6 (P6)
Other:
- note added: "NOTES:\nP6-Pin 1 EN is active low\nP6-Pin 4 CFG is not connected\nP6-Pin 5 VREF is not connected\nP6-Pin 6 SLP is active low, connected to 3V3\nP7-Pin 1 is Motor Voltage\nP7-Pin 7 FLT is not connected"
- note removed: "ChronoDot"
- moved on the sheet: C4

Commit message: Schematic, work in progress
Parts:
- removed R5, R6, R7, R8, R9: 10k, r_0805, symbol R
- removed SW2: SW_UP, SW-PB, symbol SW_PUSH
- removed SW3: SW_DN, SW-PB, symbol SW_PUSH
- removed SW4: SW_OK, SW-PB, symbol SW_PUSH
- removed SW5: SW_LT, SW-PB, symbol SW_PUSH
- removed SW6: SW_RT, SW-PB, symbol SW_PUSH
- added C11: 10uF, gearclock_fp:C_ELCO_SMD, symbol C_POL
- added C12, C13: 100nF, gearclock_fp:c_0805, symbol C_NPOL
- added C14: 100n, gearclock_fp:c_0805, symbol C
- added U5: ADXL345, gearclock_fp:ADXL345, symbol ADXL345
- B1: value I/O -> IO; footprint (none) -> gearclock_fp:IO; symbol I/O -> IO
- C1, C2, C3, C4, C6, C7: footprint ArthurC Lib:c_0805 -> gearclock_fp:c_0805
- C10, C5: footprint C4_Pretty:c_0805_led -> gearclock_fp:c_0805
- C8: footprint ArthurC Lib:C_ELCO_SMD -> gearclock_fp:C_ELCO_SMD
- LED1: footprint C4_Pretty:RGB_WS2811B -> gearclock_fp:RGB_WS2811B
- P1: footprint (none) -> gearclock_fp:Header_ISP
- P10, P8, P9: value I/O -> IO; footprint ArthurC Lib:I%2fO -> gearclock_fp:IO; symbol I/O -> IO
- P11: footprint (none) -> gearclock_fp:Pin_Header_Straight_1x09
- P12: value BAT -> 3V3_In; footprint (none) -> gearclock_fp:Pin_Header_Straight_1x02
- P13: value LiPo -> WallW; footprint (none) -> gearclock_fp:BARREL_JACK
- P2: footprint (none) -> gearclock_fp:Header_FTDI
- P3: footprint (none) -> gearclock_fp:Pin_Header_Straight_1x03
- P5: footprint (none) -> gearclock_fp:Pin_Header_Straight_1x04
- P6, P7: footprint (none) -> gearclock_fp:Pin_Header_Straight_1x08
- R1, R2, R3, R4: footprint ArthurC Lib:r_0805 -> gearclock_fp:r_0805
- SD1: footprint ArthurC Lib:SD_Micro -> gearclock_fp:SD_Micro
- SW1: footprint ArthurC Lib:SW_SMD -> gearclock_fp:Switch_SMT
- U1: footprint ArthurC Lib:TQFP32 -> gearclock_fp:TQFP32
- U2: footprint (none) -> gearclock_fp:SOT23-3
- U3: footprint ArthurC Lib:SOT23-3 -> gearclock_fp:SOT23-3
- X1: footprint ArthurC Lib:Xtal_SMD4 -> gearclock_fp:Xtal_SMD4
Connections:
- net +3.3V: now also C11.1, C12.1, C13.1, C14.1, U5.1 (VDD), U5.6 (VSS), U5.7 (CS); no longer C5.1, LED1.3 (VSS)
- net BAT: no longer C7.1, C8.1, P13.2 (P2), P7.1 (P1), U3.3 (VIN)
- net GND: now also C11.2, C12.2, C13.2, C14.2, U5.12 (SDO), U5.2 (GND), U5.4 (GND1), U5.5 (GND2)
- net SCL: now also U5.14 (SCL)
- net SDA: now also U5.13 (SDA)
- new net 5V: C5.1, C7.1, C8.1, LED1.3 (VSS), P13.2 (P2), P7.1 (P1), U3.3 (VIN)
- new net ACL_INT1: U5.8 (INT1)
- new net ACL_INT2: U5.9 (INT2)
- no-connect marks 9 -> 12
Other:
- note added: "ACCELEROMETER, I2C"
- note added: "External Wall Wart\n5V, 1A"
- note added: "NOTE:\nINT1 and INT2 - no spare pins available on uC"
- note removed: "External Battery\n3V5 min, 9V max"
- moved on the sheet: C3, C6, C7, C8, P1, P10, P11, P12, P13, P3, P5, P6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
