File: KiCAD/gearclock_rtc.sch (KiCad schematic (older format))
At the start: 7 parts, among them U4 DS3231N

Commit message: GearClock schematic needs review
Parts:
- renumbered B15 to B4, C9 to C8, R9 to R6
Changed lines of the file:
@@
 BAT
 $Comp
-L R R9
+L R R6
 U 1 1 4ECB8D22
 P 6650 2000
-F 0 "R9" V 6730 2000 50  0000 C CNN
+F 0 "R6" V 6730 2000 50  0000 C CNN
 F 1 "10k" V 6650 2000 50  0000 C CNN
 F 2 "ArthurC Lib:r_0805" H 6650 2000 60  0001 C CNN
@@
 $EndComp
 $Comp
-L +BATT #PWR09
+L +BATT #PWR08
 U 1 1 4EC101F0
 P 5300 1850
-F 0 "#PWR09" H 5300 1800 20  0001 C CNN
+F 0 "#PWR08" H 5300 1800 20  0001 C CNN
 F 1 "+BATT" H 5300 1950 30  0000 C CNN
 F 2 "" H 5300 1850 60  0001 C CNN
@@
 GND
 $Comp
-L I/O B15
+L I/O B4
 U 1 1 4E1FEBD4
 P 6825 2750
-F 0 "B15" H 6905 2750 40  0000 L CNN
+F 0 "B4" H 6905 2750 40  0000 L CNN
 F 1 "I/O" H 6825 2805 30  0001 C CNN
 F 2 "ArthurC Lib:I%2fO" H 6825 2750 60  0001 C CNN
@@
 $EndComp
 $Comp
-L C C9
+L C C8
 U 1 1 4E1FEA7E
 P 4175 2775
-F 0 "C9" H 4200 2675 50  0000 L CNN
+F 0 "C8" H 4200 2675 50  0000 L CNN
 F 1 "100n" H 4150 2375 50  0000 L CNN
 F 2 "ArthurC Lib:c_0805" H 4175 2775 60  0001 C CNN

Commit message: GearClock schematic update
Parts:
- renumbered C8 to C9, R6 to R10
Changed lines of the file:
@@
 BAT
 $Comp
-L R R6
+L R R10
 U 1 1 4ECB8D22
 P 6650 2000
-F 0 "R6" V 6730 2000 50  0000 C CNN
+F 0 "R10" V 6730 2000 50  0000 C CNN
 F 1 "10k" V 6650 2000 50  0000 C CNN
 F 2 "ArthurC Lib:r_0805" H 6650 2000 60  0001 C CNN
@@
 $EndComp
 $Comp
-L +BATT #PWR08
+L +BATT #PWR011
 U 1 1 4EC101F0
 P 5300 1850
-F 0 "#PWR08" H 5300 1800 20  0001 C CNN
+F 0 "#PWR011" H 5300 1800 20  0001 C CNN
 F 1 "+BATT" H 5300 1950 30  0000 C CNN
 F 2 "" H 5300 1850 60  0001 C CNN
@@
 $EndComp
 $Comp
-L C C8
+L C C9
 U 1 1 4E1FEA7E
 P 4175 2775
-F 0 "C8" H 4200 2675 50  0000 L CNN
+F 0 "C9" H 4200 2675 50  0000 L CNN
 F 1 "100n" H 4150 2375 50  0000 L CNN
 F 2 "ArthurC Lib:c_0805" H 4175 2775 60  0001 C CNN

Commit message: Schematic, work in progress
Parts:
- B2, B3, B4: value I/O -> IO; footprint ArthurC Lib:I%2fO -> gearclock_fp:IO; symbol I/O -> IO
- BT1: footprint ArthurC Lib:CR1632 -> gearclock_fp:CR2032
- C9: footprint ArthurC Lib:c_0805 -> gearclock_fp:c_0805
- R10: footprint ArthurC Lib:r_0805 -> gearclock_fp:r_0805
- U4: footprint ArthurC Lib:DS3231 -> gearclock_fp:DS3231
Changed lines of the file:
@@
 F 0 "R10" V 6730 2000 50  0000 C CNN
 F 1 "10k" V 6650 2000 50  0000 C CNN
-F 2 "ArthurC Lib:r_0805" H 6650 2000 60  0001 C CNN
+F 2 "gearclock_fp:r_0805" H 6650 2000 60  0001 C CNN
 F 3 "" H 6650 2000 60  0001 C CNN
 	1    6650 2000
@@
 $EndComp
 $Comp
-L +BATT #PWR10
+L +BATT #PWR014
 U 1 1 4EC101F0
 P 5300 1850
-F 0 "#PWR10" H 5300 1800 20  0001 C CNN
+F 0 "#PWR014" H 5300 1800 20  0001 C CNN
 F 1 "+BATT" H 5300 1950 30  0000 C CNN
 F 2 "" H 5300 1850 60  0001 C CNN
@@
 GND
 $Comp
-L I/O B4
+L IO B4
 U 1 1 4E1FEBD4
 P 6825 2750
 F 0 "B4" H 6905 2750 40  0000 L CNN
-F 1 "I/O" H 6825 2805 30  0001 C CNN
-F 2 "ArthurC Lib:I%2fO" H 6825 2750 60  0001 C CNN
+F 1 "IO" H 6825 2805 30  0001 C CNN
+F 2 "gearclock_fp:IO" H 6825 2750 60  0001 C CNN
 F 3 "" H 6825 2750 60  0001 C CNN
 	1    6825 2750
@@
 $EndComp
 $Comp
-L I/O B3
+L IO B3
 U 1 1 4E1FEBCE
 P 6825 2600
 F 0 "B3" H 6905 2600 40  0000 L CNN
-F 1 "I/O" H 6825 2655 30  0001 C CNN
-F 2 "ArthurC Lib:I%2fO" H 6825 2600 60  0001 C CNN
+F 1 "IO" H 6825 2655 30  0001 C CNN
+F 2 "gearclock_fp:IO" H 6825 2600 60  0001 C CNN
 F 3 "" H 6825 2600 60  0001 C CNN
 	1    6825 2600
@@
 $EndComp
 $Comp
-L I/O B2
+L IO B2
 U 1 1 4E1FEBC6
 P 6825 2450
 F 0 "B2" H 6905 2450 40  0000 L CNN
-F 1 "I/O" H 6825 2505 30  0001 C CNN
-F 2 "ArthurC Lib:I%2fO" H 6825 2450 60  0001 C CNN
+F 1 "IO" H 6825 2505 30  0001 C CNN
+F 2 "gearclock_fp:IO" H 6825 2450 60  0001 C CNN
 F 3 "" H 6825 2450 60  0001 C CNN
 	1    6825 2450
@@
 F 0 "U4" H 5850 3350 60  0000 C CNN
 F 1 "DS3231N" H 5250 2400 60  0000 C CNN
-F 2 "ArthurC Lib:DS3231" H 5550 2800 60  0001 C CNN
+F 2 "gearclock_fp:DS3231" H 5550 2800 60  0001 C CNN
 F 3 "" H 5550 2800 60  0001 C CNN
 	1    5550 2800
@@
 F 0 "C9" H 4200 2675 50  0000 L CNN
 F 1 "100n" H 4150 2375 50  0000 L CNN
-F 2 "ArthurC Lib:c_0805" H 4175 2775 60  0001 C CNN
+F 2 "gearclock_fp:c_0805" H 4175 2775 60  0001 C CNN
 F 3 "" H 4175 2775 60  0001 C CNN
 	1    4175 2775
@@
 F 0 "BT1" V 3875 2575 50  0000 C CNN
 F 1 "Batt_RTC" V 3950 2500 50  0000 C CNN
-F 2 "ArthurC Lib:CR1632" H 3950 2800 60  0001 C CNN
+F 2 "gearclock_fp:CR2032" H 3950 2800 60  0001 C CNN
 F 3 "" H 3950 2800 60  0000 C CNN
 F 4 "BU2032SM-HD-GCT-ND " H 4050 3100 60  0001 C CNN "Digikey"
